File: quad.sch (KiCad schematic (older format))
At the start: 21 parts, among them M0 Fan, M1 Fan, M2 Fan, M3 Fan, Q0 Si2318DS, Q1 Si2318DS, Q2 Si2318DS, Q4 Si2318DS

Commit message: Starting board layout
Parts:
- AE1: renamed from AE?; footprint (none) -> Connector_PinHeader_1.00mm:PinHeader_1x01_P1.00mm_Vertical
- B1: footprint RF_Mini-Circuits:Mini-Circuits_CD542_H2.84mm -> RF_Mini-Circuits:Mini-Circuits_CD541_H2.08mm
- C1: footprint (none) -> Capacitor_Tantalum_SMD:CP_EIA-7343-30_AVX-N
- C2: footprint (none) -> Capacitor_Tantalum_SMD:CP_EIA-2012-15_AVX-P
- CRF1, CRF2: footprint (none) -> Capacitor_SMD:C_0603_1608Metric
- CX1, CX2: footprint (none) -> Capacitor_SMD:C_0805_2012Metric
- JP1: renamed from JP?; footprint (none) -> Jumper:SolderJumper-3_P1.3mm_Open_Pad1.0x1.5mm
- M0, M1, M2, M3: footprint (none) -> Connector_PinSocket_2.00mm:PinSocket_1x02_P2.00mm_Vertical
- Q0, Q1, Q2, Q4: symbol Transistor_FET:Si2318DS -> quad-rescue:Si2318DS-Transistor_FET
- U3: renamed from U?; footprint (none) -> Package_DFN_QFN:QFN-64-1EP_9x9mm_P0.5mm_EP4.7x4.7mm; symbol MCU_Microchip_ATmega:ATmega256-RFR2 -> quad-rescue:ATmega256-RFR2-MCU_Microchip_ATmega
- XTAL1: footprint (none) -> Crystal:Crystal_SMD_3225-4Pin_3.2x2.5mm
- gave numbers to parts that had none: 2

Commit message: Good board outline
Parts:
- removed XTAL1: 16Mhz, Crystal:Crystal_SMD_3225-4Pin_3.2x2.5mm, symbol Device:Crystal_Small
- added Y?: Crystal_GND24_Small, symbol Device:Crystal_GND24_Small
Connections:
- net -BATT: now also Y?.2, Y?.4
- net at CX2.2, U3.56 (XTAL2): now also Y?.3
- net at CX1.2, U3.57 (XTAL1): now also Y?.1
Changed lines of the file:
@@
 	-1   0    0    1
 $EndComp
-$Comp
-L Device:Crystal_Small XTAL1
-U 1 1 5E235CEC
-P 5850 1850
-F 0 "XTAL1" H 5850 2075 50  0000 C CNN
-F 1 "16Mhz" H 5850 1984 50  0000 C CNN
-F 2 "Crystal:Crystal_SMD_3225-4Pin_3.2x2.5mm" H 5850 1850 50  0001 C CNN
-F 3 "~" H 5850 1850 50  0001 C CNN
-	1    5850 1850
-	1    0    0    -1
-$EndComp
-Wire Wire Line
-	5600 1850 5750 1850
 Wire Wire Line
 	5900 2500 5900 2000
@@
 	5900 2000 6100 2000
 Wire Wire Line
-	6100 2000 6100 1850
-Wire Wire Line
-	5600 1850 5600 2000
-Wire Wire Line
 	5600 2000 5800 2000
 Wire Wire Line
 	5800 2000 5800 2500
-Wire Wire Line
-	5950 1850 6100 1850
 $Comp
 L Device:C_Small CX1
@@
 	1    0    0    -1
 $EndComp
-Wire Wire Line
-	5600 1550 5600 1850
-Connection ~ 5600 1850
-Wire Wire Line
-	6100 1550 6100 1850
-Connection ~ 6100 1850
 Wire Wire Line
 	5600 1350 5850 1350
@@
 Wire Wire Line
 	10650 2350 10650 2400
+Wire Wire Line
+	5600 1550 5600 1750
+Wire Wire Line
+	6100 1550 6100 1750
+$Comp
+L Device:Crystal_GND24_Small Y?
+U 1 1 5E29A20B
+P 5850 1750
+F 0 "Y?" H 5994 1796 50  0000 L CNN
+F 1 "Crystal_GND24_Small" H 5994 1705 50  0000 L CNN
+F 2 "" H 5850 1750 50  0001 C CNN
+F 3 "~" H 5850 1750 50  0001 C CNN
+	1    5850 1750
+	1    0    0    -1
+$EndComp
+Wire Wire Line
+	5750 1750 5600 1750
+Connection ~ 5600 1750
+Wire Wire Line
+	5600 1750 5600 2000
+Wire Wire Line
+	5950 1750 6100 1750
+Connection ~ 6100 1750
+Wire Wire Line
+	6100 1750 6100 2000
+Wire Wire Line
+	5850 1650 5850 1350
+$Comp
+L power:VSS #PWR?
+U 1 1 5E2A0FAF
+P 5850 1900
+F 0 "#PWR?" H 5850 1750 50  0001 C CNN
+F 1 "VSS" H 5868 2073 50  0000 C CNN
+F 2 "" H 5850 1900 50  0001 C CNN
+F 3 "" H 5850 1900 50  0001 C CNN
+	1    5850 1900
+	-1   0    0    1
+$EndComp
+Wire Wire Line
+	5850 1850 5850 1900
 $EndSCHEMATC
